Commit message: updated kuka arm masses

File: drake/examples/kuka_iiwa_arm/urdf/iiwa14.urdf (robot description, URDF)
Before this commit: robot iiwa14, 11 links, 10 joints
Links:
- link iiwa_link_1: mass 4 -> 5.76
- link iiwa_link_2: mass 4 -> 6.35
- link iiwa_link_3: mass 3 -> 3.5
- link iiwa_link_4: mass 2.7 -> 3.5
- link iiwa_link_5: mass 1.7 -> 3.5
- link iiwa_link_7: mass 0.3 -> 1.2

Commit message: make torque control work on the robot with the gripper mounted, remove collision models in urdf for a faster simulation, and need to improve the gravity compensation part by using Jacobian method.

File: drake/examples/kuka_iiwa_arm/urdf/iiwa14.urdf (robot description, URDF)
Before this commit: robot iiwa14, 11 links, 10 joints
Links:
- link iiwa_link_0: geometry visual mesh filename=meshes/visual/link_0.obj
- link iiwa_link_1: geometry visual mesh filename=meshes/visual/link_1.obj
- link iiwa_link_2: geometry visual mesh filename=meshes/visual/link_2.obj
- link iiwa_link_3: geometry visual mesh filename=meshes/visual/link_3.obj
- link iiwa_link_4: geometry visual mesh filename=meshes/visual/link_4.obj
- link iiwa_link_5: geometry visual mesh filename=meshes/visual/link_5.obj
- link iiwa_link_6: geometry visual mesh filename=meshes/visual/link_6.obj

File: drake/examples/kuka_iiwa_arm/urdf/iiwa14_fixed_gripper.urdf (robot description, URDF)
Before this commit: robot iiwa14, 20 links, 19 joints
Joints:
- joint wrist: origin xyz=0 0 0 rpy=0 0 0 -> xyz=0 0 0.045 rpy=0 0 1.57; parent iiwa_link_ee_kuka -> iiwa_link_7
