Commit message: tune controller gains for grasping demo, rotate the gripper orientation

File: drake/examples/kuka_iiwa_arm/urdf/iiwa14_fixed_gripper.urdf (robot description, URDF)
Before this commit: robot iiwa14, 20 links, 19 joints
Joints:
- joint wrist: origin xyz=0 0 0.045 rpy=0 0 1.57 -> xyz=0 0 0.045 rpy=0 0 0
