Commit message: more examples edits

File: drake/examples/Valkyrie/urdf/urdf/valkyrie_simple.urdf (robot description, URDF)
Before this commit: robot valkyrie, 87 links, 86 joints
Joints:
- joint leftShoulderPitch: limit lower=-2.85 upper=2.0 effort=190 velocity=5.89 -> lower=-.75 upper=.75 effort=190 velocity=5.89; type fixed -> revolute
- joint leftShoulderRoll: origin xyz=0.0 0.2499 0.0 rpy=-1.3 0.0 0.0 -> xyz=0.0 0.2499 0.0 rpy=-1.4 0.0 0.0
- joint leftWristRoll: origin xyz=0.0 0.2871 0.0 rpy=0.0 0.0 0.0 -> xyz=0.0 0.2871 0.0 rpy=0.0 1.57 0.0
- joint rightShoulderPitch: limit lower=-2.85 upper=2.0 effort=190 velocity=5.89 -> lower=-0.75 upper=.75 effort=190 velocity=5.89; type fixed -> revolute
- joint rightShoulderRoll: origin xyz=0.0 -0.2499 0.0 rpy=1.3 0.0 0.0 -> xyz=0.0 -0.2499 0.0 rpy=1.4 0.0 0.0
- joint rightWristRoll: origin xyz=0.0 -0.2871 0.0 rpy=0.0 0.0 0.0 -> xyz=0.0 -0.2871 0.0 rpy=0 1.57 0
