Commit message: initialization

File: drake/examples/KukaArm/urdf/iiwa14_fixed_gripper.urdf (robot description, URDF)
Before this commit: robot iiwa14, 14 links, 12 joints
Joints:
- added joint gripper_base_joint: type fixed, parent base_link, child right_finger, origin xyz=0 0.04 0.0375 rpy=0 0 0
- joint base_joint: child right_finger -> iiwa_link_0; origin xyz=0 0.04 0.0375 rpy=0 0 0 -> xyz=0 0 0.0 rpy=0 0 0; parent base_link -> base

Commit message: add passive forward simulation

File: drake/examples/KukaArm/urdf/iiwa14_fixed_gripper.urdf (robot description, URDF)
Before this commit: robot iiwa14, 14 links, 13 joints
Links:
- link left_finger: geometry collision sphere radius=0.0; collision sphere radius=0.0
- link right_finger: geometry collision sphere radius=0.0; collision sphere radius=0.0
